File: external_conn.sch (KiCad schematic (older format))
At the start: 0 parts

Commit message: Various components added
USB conn, general outputs, brake signal, touch sensor
Parts:
- added U?: CONN_USB, symbol CONN_USB
Changed lines of the file:
@@
 $Descr A4 11693 8268
 encoding utf-8
-Sheet 1 14
+Sheet 5 11
 Title ""
 Date "10 nov 2013"
@@
 Comment4 ""
 $EndDescr
+$Comp
+L CONN_USB U?
+U 1 1 52807223
+P 850 550
+F 0 "U?" H 850 550 60  0000 C CNN
+F 1 "CONN_USB" H 850 -100 60  0000 C CNN
+F 2 "" H 850 550 60  0000 C CNN
+F 3 "" H 850 550 60  0000 C CNN
+	1    850  550
+	1    0    0    -1
+$EndComp
 $EndSCHEMATC
