File: battery_pack.sch (KiCad schematic (older format))
At the start: 0 parts

Commit message: Various components added
USB conn, general outputs, brake signal, touch sensor
Parts:
- added BT?: BATTERY, ~, symbol BATTERY
- added D?: SCHDPAK, ~, symbol SCHDPAK
- added D?: DOUBLE_SCHOTTKY, ~, symbol DOUBLE_SCHOTTKY
- added R?: 1.58M, ~, symbol R
- added R?: 102K, ~, symbol R
- added R?: 191K, ~, symbol R
- added R? (x2): Nominal, ~, symbol R
- added U?: TPS3700, symbol TPS3700
- added U? (x2): 74LVC2G06, symbol 74LVC2G06
- added U? (x2): NC7WZ08, symbol NC7WZ08
Connections:
- net labels added: +3.3V, CHG, DGND, NMOS_CTRL, PMOS_CTRL, V_BATT, ~CHG, ~OV, ~UV
- wire segments 0 -> 37

Commit message: Battery management stuff
:D
Parts:
- removed BT?: BATTERY, ~, symbol BATTERY
- removed D?: SCHDPAK, ~, symbol SCHDPAK
- removed D?: DOUBLE_SCHOTTKY, ~, symbol DOUBLE_SCHOTTKY
- removed R?: 1.58M, ~, symbol R
- removed R?: 102K, ~, symbol R
- removed R?: 191K, ~, symbol R
- removed R? (x2): Nominal, ~, symbol R
- removed U?: TPS3700, symbol TPS3700
- removed U? (x2): 74LVC2G06, symbol 74LVC2G06
- removed U? (x2): NC7WZ08, symbol NC7WZ08
- added C? (x2): Cap Steadystate, ~, symbol C
- added F?: FUSE, ~, symbol FUSE
- added R?: R, ~, symbol R
- added U? (x2): MCP6L02, symbol MCP6L02
Connections:
- net labels added: V_PACK, V_PACK_BUFFERED
- net labels removed: CHG, NMOS_CTRL, PMOS_CTRL, V_BATT, ~CHG, ~OV, ~UV
- wire segments 37 -> 36

Commit message: random minor thing
Other:
- note added: "Should we include a fuse?"
- note added: "What should the current sense resistor be?"
Changed lines of the file:
@@
 Sheet 2 14
 Title ""
-Date "12 nov 2013"
+Date "15 nov 2013"
 Rev ""
 Comp ""
@@
 Wire Wire Line
 	3250 1950 3250 2000
+Text Notes 650  700  0    60   ~ 0
+Should we include a fuse?
+Text Notes 650  1050 0    60   ~ 0
+What should the current sense resistor be?
 $EndSCHEMATC
