File: output_signal_brake_2.sch (KiCad schematic (older format))
At the start: 50 parts

Commit message: uh. same as before? some glitch
Connections:
- net labels added: +2.5V local
- net labels removed: +2.5V
- wire segments 133 -> 193
Changed lines of the file:
@@
 Sheet 15 18
 Title ""
-Date "12 dec 2013"
+Date "13 dec 2013"
 Rev ""
 Comp ""
@@
 	2650 1400 2650 1750
 Wire Wire Line
-	1500 1400 2800 1400
+	1700 1400 1750 1400
+Wire Wire Line
+	1750 1400 1900 1400
+Wire Wire Line
+	1900 1400 2050 1400
+Wire Wire Line
+	2050 1400 2200 1400
+Wire Wire Line
+	2200 1400 2350 1400
+Wire Wire Line
+	2350 1400 2500 1400
+Wire Wire Line
+	2500 1400 2650 1400
+Wire Wire Line
+	2650 1400 2800 1400
 Wire Wire Line
 	2350 1400 2350 1750
@@
 	9050 1400 9050 1750
 Wire Wire Line
-	9400 1650 9950 1650
-Wire Wire Line
-	9400 1400 9400 1750
+	9400 1650 9700 1650
+Wire Wire Line
+	9700 1650 9950 1650
+Wire Wire Line
+	9400 1400 9400 1650
+Wire Wire Line
+	9400 1650 9400 1750
 Wire Wire Line
 	9700 1750 9700 1650
 Connection ~ 9700 1650
 Wire Wire Line
-	9350 2150 9950 2150
+	9350 2150 9400 2150
+Wire Wire Line
+	9400 2150 9700 2150
+Wire Wire Line
+	9700 2150 9950 2150
 Connection ~ 9700 2150
 Connection ~ 9400 1650
@@
 	9200 1800 9200 2250
 Wire Wire Line
-	10250 1400 10250 1750
-Wire Wire Line
-	10250 1650 10750 1650
-Wire Wire Line
-	10250 2150 10750 2150
+	10250 1400 10250 1650
+Wire Wire Line
+	10250 1650 10250 1750
+Wire Wire Line
+	10250 1650 10500 1650
+Wire Wire Line
+	10500 1650 10750 1650
+Wire Wire Line
+	10250 2150 10500 2150
+Wire Wire Line
+	10500 2150 10750 2150
 Connection ~ 10250 1650
 Wire Wire Line
-	8200 1400 10250 1400
+	8400 1400 8450 1400
+Wire Wire Line
+	8450 1400 8600 1400
+Wire Wire Line
+	8600 1400 8750 1400
+Wire Wire Line
+	8750 1400 8900 1400
+Wire Wire Line
+	8900 1400 9050 1400
+Wire Wire Line
+	9050 1400 9200 1400
+Wire Wire Line
+	9200 1400 9400 1400
+Wire Wire Line
+	9400 1400 10250 1400
 Connection ~ 8450 1400
 Connection ~ 8600 1400
@@
 	5700 1400 5700 1750
 Wire Wire Line
-	6050 1650 6600 1650
-Wire Wire Line
-	6050 1400 6050 1750
+	6050 1650 6350 1650
+Wire Wire Line
+	6350 1650 6600 1650
+Wire Wire Line
+	6050 1400 6050 1650
+Wire Wire Line
+	6050 1650 6050 1750
 Wire Wire Line
 	6350 1750 6350 1650
 Connection ~ 6350 1650
 Wire Wire Line
-	6000 2150 6600 2150
+	6000 2150 6050 2150
+Wire Wire Line
+	6050 2150 6350 2150
+Wire Wire Line
+	6350 2150 6600 2150
 Connection ~ 6350 2150
 Connection ~ 6050 1650
@@
 	5850 1800 5850 2250
 Wire Wire Line
-	6900 1400 6900 1750
-Wire Wire Line
-	6900 1650 7400 1650
-Wire Wire Line
-	6900 2150 7400 2150
+	6900 1400 6900 1650
+Wire Wire Line
+	6900 1650 6900 1750
+Wire Wire Line
+	6900 1650 7150 1650
+Wire Wire Line
+	7150 1650 7400 1650
+Wire Wire Line
+	6900 2150 7150 2150
+Wire Wire Line
+	7150 2150 7400 2150
 Connection ~ 6900 1650
 Wire Wire Line
-	4850 1400 6900 1400
+	5050 1400 5100 1400
+Wire Wire Line
+	5100 1400 5250 1400
+Wire Wire Line
+	5250 1400 5400 1400
+Wire Wire Line
+	5400 1400 5550 1400
+Wire Wire Line
+	5550 1400 5700 1400
+Wire Wire Line
+	5700 1400 5850 1400
+Wire Wire Line
+	5850 1400 6050 1400
+Wire Wire Line
+	6050 1400 6900 1400
 Connection ~ 5100 1400
 Connection ~ 5250 1400
@@
 	900  3050 1000 3050
 Wire Wire Line
-	4350 3200 4350 3500
+	4350 3200 4350 3300
+Wire Wire Line
+	4350 3300 4350 3400
+Wire Wire Line
+	4350 3400 4350 3500
 Connection ~ 4350 3300
 Connection ~ 4350 3400
 Wire Wire Line
-	1000 3200 1000 3500
+	1000 3200 1000 3300
+Wire Wire Line
+	1000 3300 1000 3400
+Wire Wire Line
+	1000 3400 1000 3500
 Connection ~ 1000 3300
 Connection ~ 1000 3400
 Wire Wire Line
-	7700 3200 7700 3500
+	7700 3200 7700 3300
+Wire Wire Line
+	7700 3300 7700 3400
+Wire Wire Line
+	7700 3400 7700 3500
 Connection ~ 7700 3300
 Connection ~ 7700 3400
@@
 	6550 3400 6600 3400
 Wire Wire Line
-	7100 2900 7100 3500
+	7100 2900 7100 3100
+Wire Wire Line
+	7100 3100 7100 3200
+Wire Wire Line
+	7100 3200 7100 3400
+Wire Wire Line
+	7100 3400 7100 3500
 Wire Wire Line
 	9900 3400 9950 3400
@@
 	3200 3400 3250 3400
 Wire Wire Line
-	3750 3000 3750 3500
+	3750 3000 3750 3100
+Wire Wire Line
+	3750 3100 3750 3200
+Wire Wire Line
+	3750 3200 3750 3400
+Wire Wire Line
+	3750 3400 3750 3500
 Wire Wire Line
 	3200 3000 3750 3000
@@
 $EndComp
 Wire Wire Line
-	10450 3100 10450 3500
+	10450 3100 10450 3200
+Wire Wire Line
+	10450 3200 10450 3400
+Wire Wire Line
+	10450 3400 10450 3500
 Wire Wire Line
 	9900 3100 10450 3100
 Wire Wire Line
-	9950 2800 9950 3000
+	9950 2800 9950 2900
+Wire Wire Line
+	9950 2900 9950 3000
 Wire Wire Line
 	9950 3000 9900 3000
@@
 $EndComp
 Wire Wire Line
-	8350 5250 8500 5250
+	8350 5250 8450 5250
+Wire Wire Line
+	8450 5250 8500 5250
 Wire Wire Line
 	8450 5250 8450 5400
@@
 Connection ~ 8450 5250
 Wire Wire Line
-	9100 5250 10050 5250
+	9100 5250 9150 5250
+Wire Wire Line
+	9150 5250 9400 5250
+Wire Wire Line
+	9400 5250 9650 5250
+Wire Wire Line
+	9650 5250 9900 5250
+Wire Wire Line
+	9900 5250 10150 5250
 Wire Wire Line
 	9400 5250 9400 5300
@@
 Connection ~ 9900 5250
 Wire Wire Line
-	9400 5500 9400 5600
+	9400 5500 9400 5550
+Wire Wire Line
+	9400 5550 9400 5600
 Wire Wire Line
 	8350 5550 9150 5550
@@
 	9100 5850 9100 6050
 Wire Wire Line
-	9100 6050 10050 6050
-Wire Wire Line
-	6250 5250 6850 5250
+	9100 6050 9650 6050
+Wire Wire Line
+	9650 6050 10050 6050
+Wire Wire Line
+	6250 5250 6400 5250
+Wire Wire Line
+	6400 5250 6850 5250
 Wire Wire Line
 	6400 5300 6400 5250
@@
 Wire Wire Line
 	9900 5500 9900 5550
-$Comp
-L +2.5V #PWR?
-U 1 1 52A6A9DD
-P 10050 5200
-F 0 "#PWR?" H 10050 5150 20  0001 C CNN
-F 1 "+2.5V" H 10050 5300 30  0000 C CNN
-F 2 "" H 10050 5200 60  0000 C CNN
-F 3 "" H 10050 5200 60  0000 C CNN
-	1    10050 5200
-	1    0    0    -1
-$EndComp
-Wire Wire Line
-	10050 5250 10050 5200
 Text Notes 6800 4750 0    60   ~ 0
 Battery to 2.5V Buck Power Supply
@@
 Connection ~ 9650 6050
 Wire Wire Line
-	7500 6600 8350 6600
+	7500 6600 7600 6600
+Wire Wire Line
+	7600 6600 7700 6600
+Wire Wire Line
+	7700 6600 8350 6600
 Connection ~ 7700 6600
 Connection ~ 7600 6600
@@
 $EndComp
 $Comp
-L +2.5V #PWR?
-U 1 1 52A802AB
-P 1500 1400
-F 0 "#PWR?" H 1500 1350 20  0001 C CNN
-F 1 "+2.5V" H 1500 1500 30  0000 C CNN
-F 2 "" H 1500 1400 60  0000 C CNN
-F 3 "" H 1500 1400 60  0000 C CNN
-	1    1500 1400
-	1    0    0    -1
-$EndComp
-$Comp
-L +2.5V #PWR?
-U 1 1 52A802B1
-P 4850 1400
-F 0 "#PWR?" H 4850 1350 20  0001 C CNN
-F 1 "+2.5V" H 4850 1500 30  0000 C CNN
-F 2 "" H 4850 1400 60  0000 C CNN
-F 3 "" H 4850 1400 60  0000 C CNN
-	1    4850 1400
-	1    0    0    -1
-$EndComp
-$Comp
-L +2.5V #PWR?
-U 1 1 52A802B7
-P 8200 1400
-F 0 "#PWR?" H 8200 1350 20  0001 C CNN
-F 1 "+2.5V" H 8200 1500 30  0000 C CNN
-F 2 "" H 8200 1400 60  0000 C CNN
-F 3 "" H 8200 1400 60  0000 C CNN
-	1    8200 1400
-	1    0    0    -1
-$EndComp
-$Comp
 L R R?
 U 1 1 52A80325
@@
 PWR_GOOD
 Wire Wire Line
-	6850 5250 6850 5550
+	6850 5250 6850 5400
+Wire Wire Line
+	6850 5400 6850 5550
 Connection ~ 6850 5400
 Text HLabel 6250 5700 0    60   Input ~ 0
@@
 Wire Wire Line
 	6250 5700 6850 5700
+Text Label 10150 5250 0    60   ~ 0
++2.5V local
+Text Label 1700 1400 2    60   ~ 0
++2.5V local
+Text Label 5050 1400 2    60   ~ 0
++2.5V local
+Text Label 8400 1400 2    60   ~ 0
++2.5V local
 $EndSCHEMATC

Commit message: added pullups/downs as necessary, added test pts
also added interrupt conn to msp from charger, made led part for generic
indicators, added generic indicators to psu's
Parts:
- removed R?: Nominal, ~, symbol R
- added C?: Cap Nominal, ~, symbol C
- added D?: LED_GENERIC_SMD, ~, symbol LED_GENERIC_SMD
- added R? (x2): Nominal, ~, symbol R
- added R?: 300, ~, symbol R
Connections:
- wire segments 193 -> 139
Other:
- note added: "1.9V @ 2mA"
- note added: "Indicator LED"
- note removed: "Don't think we need this output\nor the pull up here. We aren't reading it...?"

Commit message: various fixes due to issues found in ERC
learned how to use invisible pins
Parts:
- gave numbers to parts that had none: 54

Commit message: placed components ... quite the task!
there is a lot of shit going on in this board... :D
Parts:
- renumbered C22 to C17, C23 to C18, C24 to C19, C25 to C20, C26 to C21, C27 to C22, C28 to C23, C29 to C24, D36 to D10, D37 to D11, D38 to D12, D39 to D13, D40 to D14, D41 to D15, D42 to D16, D43 to D17, D44 to D18, D45 to D19, D46 to D20, D47 to D21, D48 to D22, D49 to D23, D50 to D24, D51 to D25, D52 to D26, D53 to D27, D54 to D28, D55 to D29, D56 to D30, D57 to D31, D58 to D32, D59 to D33, D60 to D34, D61 to D35, D62 to D36, R36 to R31, R37 to R32, R38 to R33, R39 to R34, R40 to R35, R41 to R36, R42 to R37, R43 to R38, R44 to R39, R45 to R40, R46 to R41, R47 to R42, R48 to R43, R49 to R44, U42 to U39, U43 to U40, U44 to U41, U45 to U42

Commit message: revisions to board and sch
Parts:
- removed D10, D11, D12, D13, D20, D21, D22, D23: LS-E63F, ~, symbol LS-E63F
- removed D14, D15, D16, D17, D18, D19, D24, D25, D26, D30, D31, D32: LY-E63F, ~, symbol LY-E63F
- removed D27, D28, D33, D34: LY-A67F, ~, symbol LY-A67F
- removed D29, D35: LR-A67F, ~, symbol LR-A67F
- removed R31, R32, R33, R34, R35, R36: 200, ~, symbol R
- added P1, P3, P4: CONN_6_RA_MALE, symbol CONN_6
- added P2: CONN_6_RA_FEMALE, symbol CONN_6
- added P5: CONN_6_MALE_FRONT, symbol CONN_6
- added P6: CONN_6_MALE_BACK, symbol CONN_6
Connections:
- wire segments 139 -> 183
- no-connect marks 42 -> 36
Other:
- note removed: "Front Turn Signal"
- note removed: "Rear Brake"
- note removed: "Rear Turn Signal"
- note removed: "Side Brake"
- note removed: "Side Turn Signal"
- moved on the sheet: C17, C18, C19, C20, D36, R37, R38, R39, R40, R42, U39, U40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
