File: battery_charger.sch (KiCad schematic (older format))
At the start: 23 parts, among them U52 BQ24190

Commit message: placed components ... quite the task!
there is a lot of shit going on in this board... :D
Parts:
- renumbered C37 to C31, C38 to C32, C39 to C33, C40 to C34, C41 to C35, C42 to C36, C43 to C37, D65 to D38, R53 to R48, R54 to R49, R55 to R50, R56 to R51, R57 to R52, R58 to R53, R59 to R54, R60 to R55, R61 to R56, R62 to R57, R63 to R58, U52 to U48
Changed lines of the file:
@@
 $Descr A4 11693 8268
 encoding utf-8
-Sheet 18 18
+Sheet 18 15
 Title ""
-Date "12 jan 2014"
+Date "18 jan 2014"
 Rev ""
 Comp ""
@@
 USB_D-
 $Comp
-L DGND #PWR0124
+L DGND #PWR0110
 U 1 1 5292B82E
 P 3600 3400
-F 0 "#PWR0124" H 3600 3400 40  0001 C CNN
+F 0 "#PWR0110" H 3600 3400 40  0001 C CNN
 F 1 "DGND" H 3600 3330 40  0000 C CNN
 F 2 "" H 3600 3400 60  0000 C CNN
@@
 $EndComp
 $Comp
-L R R55
+L R R50
 U 1 1 5292B87D
 P 3050 2100
-F 0 "R55" V 3130 2100 40  0000 C CNN
+F 0 "R50" V 3130 2100 40  0000 C CNN
 F 1 "Nominal" V 3057 2101 40  0000 C CNN
 F 2 "~" V 2980 2100 30  0000 C CNN
@@
 $EndComp
 $Comp
-L R R56
+L R R51
 U 1 1 5292B883
 P 3250 2100
-F 0 "R56" V 3330 2100 40  0000 C CNN
+F 0 "R51" V 3330 2100 40  0000 C CNN
 F 1 "Nominal" V 3257 2101 40  0000 C CNN
 F 2 "~" V 3180 2100 30  0000 C CNN
@@
 $EndComp
 $Comp
-L R R57
+L R R52
 U 1 1 5292B889
 P 3450 2100
-F 0 "R57" V 3530 2100 40  0000 C CNN
+F 0 "R52" V 3530 2100 40  0000 C CNN
 F 1 "Nominal" V 3457 2101 40  0000 C CNN
 F 2 "~" V 3380 2100 30  0000 C CNN
@@
 $EndComp
 $Comp
-L R R58
+L R R53
 U 1 1 5292B88F
 P 5750 3050
-F 0 "R58" V 5830 3050 40  0000 C CNN
+F 0 "R53" V 5830 3050 40  0000 C CNN
 F 1 "5.52K" V 5757 3051 40  0000 C CNN
 F 2 "~" V 5680 3050 30  0000 C CNN
@@
 $EndComp
 $Comp
-L R R62
+L R R57
 U 1 1 5292B895
 P 5750 3650
-F 0 "R62" V 5830 3650 40  0000 C CNN
+F 0 "R57" V 5830 3650 40  0000 C CNN
 F 1 "31.23K" V 5757 3651 40  0000 C CNN
 F 2 "~" V 5680 3650 30  0000 C CNN
@@
 $EndComp
 $Comp
-L R R59
+L R R54
 U 1 1 5292B89B
 P 6400 3050
-F 0 "R59" V 6480 3050 40  0000 C CNN
+F 0 "R54" V 6480 3050 40  0000 C CNN
 F 1 "5.52K" V 6407 3051 40  0000 C CNN
 F 2 "~" V 6330 3050 30  0000 C CNN
@@
 $EndComp
 $Comp
-L R R63
+L R R58
 U 1 1 5292B8A1
 P 6400 3650
-F 0 "R63" V 6480 3650 40  0000 C CNN
+F 0 "R58" V 6480 3650 40  0000 C CNN
 F 1 "31.23K" V 6407 3651 40  0000 C CNN
 F 2 "~" V 6330 3650 30  0000 C CNN
@@
 $EndComp
 $Comp
-L R R60
+L R R55
 U 1 1 5292B8A7
 P 3850 3300
-F 0 "R60" V 3930 3300 40  0000 C CNN
+F 0 "R55" V 3930 3300 40  0000 C CNN
 F 1 "267" V 3857 3301 40  0000 C CNN
 F 2 "~" V 3780 3300 30  0000 C CNN
@@
 $EndComp
 $Comp
-L BQ24190 U52
+L BQ24190 U48
 U 1 1 52A98672
 P 4800 1650
-F 0 "U52" H 4800 1650 60  0000 C CNN
+F 0 "U48" H 4800 1650 60  0000 C CNN
 F 1 "BQ24190" H 4800 -200 60  0000 C CNN
 F 2 "~" H 4800 1650 60  0000 C CNN
@@
 $EndComp
 $Comp
-L DGND #PWR0125
+L DGND #PWR0111
 U 1 1 52A986BA
 P 5400 3500
-F 0 "#PWR0125" H 5400 3500 40  0001 C CNN
+F 0 "#PWR0111" H 5400 3500 40  0001 C CNN
 F 1 "DGND" H 5400 3430 40  0000 C CNN
 F 2 "" H 5400 3500 60  0000 C CNN
@@
 	5750 3900 6700 3900
 $Comp
-L DGND #PWR0126
+L DGND #PWR0112
 U 1 1 52A98A95
 P 5750 4000
-F 0 "#PWR0126" H 5750 4000 40  0001 C CNN
+F 0 "#PWR0112" H 5750 4000 40  0001 C CNN
 F 1 "DGND" H 5750 3930 40  0000 C CNN
 F 2 "" H 5750 4000 60  0000 C CNN
@@
 	4200 1400 4200 1850
 $Comp
-L C C37
+L C C31
 U 1 1 52AAD29A
 P 3950 1600
-F 0 "C37" H 3950 1700 40  0000 L CNN
+F 0 "C31" H 3950 1700 40  0000 L CNN
 F 1 "1uF" H 3956 1515 40  0000 L CNN
 F 2 "~" H 3988 1450 30  0000 C CNN
@@
 Connection ~ 3950 1400
 $Comp
-L DGND #PWR0127
+L DGND #PWR0113
 U 1 1 52AAD37B
 P 3950 1850
-F 0 "#PWR0127" H 3950 1850 40  0001 C CNN
+F 0 "#PWR0113" H 3950 1850 40  0001 C CNN
 F 1 "DGND" H 3950 1780 40  0000 C CNN
 F 2 "" H 3950 1850 60  0000 C CNN
@@
 	3750 1500 1900 1500
 $Comp
-L +3.3V #PWR0128
+L +3.3V #PWR0114
 U 1 1 52AAD3EE
 P 2850 1750
-F 0 "#PWR0128" H 2850 1710 30  0001 C CNN
+F 0 "#PWR0114" H 2850 1710 30  0001 C CNN
 F 1 "+3.3V" H 2850 1860 30  0000 C CNN
 F 2 "" H 2850 1750 60  0000 C CNN
@@
 Connection ~ 3250 1850
 $Comp
-L C C38
+L C C32
 U 1 1 52AAD4A2
 P 1900 1700
-F 0 "C38" H 1900 1800 40  0000 L CNN
+F 0 "C32" H 1900 1800 40  0000 L CNN
 F 1 "6.8uF" H 1906 1615 40  0000 L CNN
 F 2 "~" H 1938 1550 30  0000 C CNN
@@
 $EndComp
 $Comp
-L DGND #PWR0129
+L DGND #PWR0115
 U 1 1 52AAD4B3
 P 1900 1950
-F 0 "#PWR0129" H 1900 1950 40  0001 C CNN
+F 0 "#PWR0115" H 1900 1950 40  0001 C CNN
 F 1 "DGND" H 1900 1880 40  0000 C CNN
 F 2 "" H 1900 1950 60  0000 C CNN
@@
 	2050 3150 4200 3150
 $Comp
-L C C42
+L C C36
 U 1 1 52AB375A
 P 6950 2800
-F 0 "C42" H 6950 2900 40  0000 L CNN
+F 0 "C36" H 6950 2900 40  0000 L CNN
 F 1 "10uF" H 6956 2715 40  0000 L CNN
 F 2 "~" H 6988 2650 30  0000 C CNN
@@
 $EndComp
 $Comp
-L DGND #PWR0130
+L DGND #PWR0116
 U 1 1 52AB3760
 P 6950 3050
-F 0 "#PWR0130" H 6950 3050 40  0001 C CNN
+F 0 "#PWR0116" H 6950 3050 40  0001 C CNN
 F 1 "DGND" H 6950 2980 40  0000 C CNN
 F 2 "" H 6950 3050 60  0000 C CNN
@@
 Connection ~ 6950 2600
 $Comp
-L C C39
+L C C33
 U 1 1 52AB388A
 P 5600 1850
-F 0 "C39" H 5600 1950 40  0000 L CNN
+F 0 "C33" H 5600 1950 40  0000 L CNN
 F 1 "47nF" H 5606 1765 40  0000 L CNN
 F 2 "~" H 5638 1700 30  0000 C CNN
@@
 Connection ~ 6400 2800
 $Comp
-L C C43
+L C C37
 U 1 1 52AB3E00
 P 6650 3000
-F 0 "C43" H 6650 3100 40  0000 L CNN
+F 0 "C37" H 6650 3100 40  0000 L CNN
 F 1 "4.7uF" H 6656 2915 40  0000 L CNN
 F 2 "~" H 6688 2850 30  0000 C CNN
@@
 $EndComp
 $Comp
-L DGND #PWR0131
+L DGND #PWR0117
 U 1 1 52AB3E06
 P 6650 3250
-F 0 "#PWR0131" H 6650 3250 40  0001 C CNN
+F 0 "#PWR0117" H 6650 3250 40  0001 C CNN
 F 1 "DGND" H 6650 3180 40  0000 C CNN
 F 2 "" H 6650 3250 60  0000 C CNN
@@
 Connection ~ 6400 1650
 $Comp
-L C C40
+L C C34
 U 1 1 52AB3EAE
 P 6650 1850
-F 0 "C40" H 6650 1950 40  0000 L CNN
+F 0 "C34" H 6650 1950 40  0000 L CNN
 F 1 "10uF" H 6656 1765 40  0000 L CNN
 F 2 "~" H 6688 1700 30  0000 C CNN
@@
 $EndComp
 $Comp
-L DGND #PWR0132
+L DGND #PWR0118
 U 1 1 52AB3EB4
 P 6650 2100
-F 0 "#PWR0132" H 6650 2100 40  0001 C CNN
+F 0 "#PWR0118" H 6650 2100 40  0001 C CNN
 F 1 "DGND" H 6650 2030 40  0000 C CNN
 F 2 "" H 6650 2100 60  0000 C CNN
@@
 	6650 2050 6650 2100
 $Comp
-L C C41
+L C C35
 U 1 1 52AB3EBB
 P 6950 1850
-F 0 "C41" H 6950 1950 40  0000 L CNN
+F 0 "C35" H 6950 1950 40  0000 L CNN
 F 1 "10uF" H 6956 1765 40  0000 L CNN
 F 2 "~" H 6988 1700 30  0000 C CNN
@@
 $EndComp
 $Comp
-L DGND #PWR0133
+L DGND #PWR0119
 U 1 1 52AB3EC1
 P 6950 2100
-F 0 "#PWR0133" H 6950 2100 40  0001 C CNN
+F 0 "#PWR0119" H 6950 2100 40  0001 C CNN
 F 1 "DGND" H 6950 2030 40  0000 C CNN
 F 2 "" H 6950 2100 60  0000 C CNN
@@
 Indicator LED
 $Comp
-L LED_GENERIC_SMD D65
+L LED_GENERIC_SMD D38
 U 1 1 52B37BFF
 P 2450 3450
-F 0 "D65" H 2450 3550 50  0000 C CNN
+F 0 "D38" H 2450 3550 50  0000 C CNN
 F 1 "LED_GENERIC_SMD" H 2450 3300 50  0001 C CNN
 F 2 "~" H 2450 3450 60  0000 C CNN
@@
 1.9V @ 2mA
 $Comp
-L DGND #PWR0134
+L DGND #PWR0120
 U 1 1 52B37C0F
 P 2450 3800
-F 0 "#PWR0134" H 2450 3800 40  0001 C CNN
+F 0 "#PWR0120" H 2450 3800 40  0001 C CNN
 F 1 "DGND" H 2450 3730 40  0000 C CNN
 F 2 "" H 2450 3800 60  0000 C CNN
@@
 Connection ~ 2850 1850
 $Comp
-L R R54
+L R R49
 U 1 1 52B3B9CF
 P 2850 2100
-F 0 "R54" V 2930 2100 40  0000 C CNN
+F 0 "R49" V 2930 2100 40  0000 C CNN
 F 1 "Nominal" V 2857 2101 40  0000 C CNN
 F 2 "~" V 2780 2100 30  0000 C CNN
@@
 Connection ~ 2850 2850
 $Comp
-L R R53
+L R R48
 U 1 1 52B3BA8E
 P 2450 2100
-F 0 "R53" V 2530 2100 40  0000 C CNN
+F 0 "R48" V 2530 2100 40  0000 C CNN
 F 1 "700" V 2457 2101 40  0000 C CNN
 F 2 "~" V 2380 2100 30  0000 C CNN
@@
 Connection ~ 2650 2950
 $Comp
-L R R61
+L R R56
 U 1 1 52B3BBFD
 P 2650 3500
-F 0 "R61" V 2730 3500 40  0000 C CNN
+F 0 "R56" V 2730 3500 40  0000 C CNN
 F 1 "Nominal" V 2657 3501 40  0000 C CNN
 F 2 "~" V 2580 3500 30  0000 C CNN
