File: battery_module.sch (KiCad schematic (older format))
At the start: 12 parts, among them Q1 AON7611, U21 74LVC2G06, U22 TPS3700, U23 NC7WZ08

Commit message: placed components ... quite the task!
there is a lot of shit going on in this board... :D
Changed lines of the file:
@@
 $Descr A4 11693 8268
 encoding utf-8
-Sheet 3 18
+Sheet 3 15
 Title ""
-Date "12 jan 2014"
+Date "18 jan 2014"
 Rev ""
 Comp ""
@@
 AR Path="/5224C457/5281E180/5281D336" Ref="BT2"  Part="1"
 AR Path="/5224C457/5281E2A4/5281D336" Ref="BT3"  Part="1"
-F 0 "BT1" H 1300 2000 50  0000 C CNN
+F 0 "BT3" H 1300 2000 50  0000 C CNN
 F 1 "BATTERY" H 1300 1610 50  0000 C CNN
 F 2 "~" H 1300 1800 60  0000 C CNN
@@
 AR Path="/5224C457/5281E180/5281D33C" Ref="U25"  Part="1"
 AR Path="/5224C457/5281E2A4/5281D33C" Ref="U28"  Part="1"
-F 0 "U22" H 2450 2150 60  0000 C CNN
+F 0 "U28" H 2450 2150 60  0000 C CNN
 F 1 "TPS3700" H 2450 1550 60  0000 C CNN
 F 2 "" H 2450 2100 60  0000 C CNN
@@
 AR Path="/5224C457/5281E180/5281D342" Ref="R7"  Part="1"
 AR Path="/5224C457/5281E2A4/5281D342" Ref="R12"  Part="1"
-F 0 "R2" V 1780 1750 40  0000 C CNN
+F 0 "R12" V 1780 1750 40  0000 C CNN
 F 1 "1.58M" V 1707 1751 40  0000 C CNN
 F 2 "~" V 1630 1750 30  0000 C CNN
@@
 AR Path="/5224C457/5281E180/5281D348" Ref="R10"  Part="1"
 AR Path="/5224C457/5281E2A4/5281D348" Ref="R15"  Part="1"
-F 0 "R5" V 1780 2350 40  0000 C CNN
+F 0 "R15" V 1780 2350 40  0000 C CNN
 F 1 "102K" V 1707 2351 40  0000 C CNN
 F 2 "~" V 1630 2350 30  0000 C CNN
@@
 AR Path="/5224C457/5281E180/5281D34E" Ref="R11"  Part="1"
 AR Path="/5224C457/5281E2A4/5281D34E" Ref="R16"  Part="1"
-F 0 "R6" V 1780 2950 40  0000 C CNN
+F 0 "R16" V 1780 2950 40  0000 C CNN
 F 1 "191K" V 1707 2951 40  0000 C CNN
 F 2 "~" V 1630 2950 30  0000 C CNN
@@
 $EndComp
 $Comp
-L DGND #PWR08
+L DGND #PWR06
 U 1 1 5281D354
 P 1700 3250
-AR Path="/5224C457/5281D330/5281D354" Ref="#PWR08"  Part="1"
-AR Path="/5224C457/5281E180/5281D354" Ref="#PWR017"  Part="1"
-AR Path="/5224C457/5281E2A4/5281D354" Ref="#PWR026"  Part="1"
-F 0 "#PWR08" H 1700 3250 40  0001 C CNN
+AR Path="/5224C457/5281D330/5281D354" Ref="#PWR06"  Part="1"
+AR Path="/5224C457/5281E180/5281D354" Ref="#PWR015"  Part="1"
+AR Path="/5224C457/5281E2A4/5281D354" Ref="#PWR024"  Part="1"
+F 0 "#PWR024" H 1700 3250 40  0001 C CNN
 F 1 "DGND" H 1700 3180 40  0000 C CNN
 F 2 "" H 1700 3250 60  0000 C CNN
@@
 $EndComp
 $Comp
-L DGND #PWR09
+L DGND #PWR07
 U 1 1 5281D35A
 P 1300 2150
-AR Path="/5224C457/5281D330/5281D35A" Ref="#PWR09"  Part="1"
-AR Path="/5224C457/5281E180/5281D35A" Ref="#PWR018"  Part="1"
-AR Path="/5224C457/5281E2A4/5281D35A" Ref="#PWR027"  Part="1"
-F 0 "#PWR09" H 1300 2150 40  0001 C CNN
+AR Path="/5224C457/5281D330/5281D35A" Ref="#PWR07"  Part="1"
+AR Path="/5224C457/5281E180/5281D35A" Ref="#PWR016"  Part="1"
+AR Path="/5224C457/5281E2A4/5281D35A" Ref="#PWR025"  Part="1"
+F 0 "#PWR025" H 1300 2150 40  0001 C CNN
 F 1 "DGND" H 1300 2080 40  0000 C CNN
 F 2 "" H 1300 2150 60  0000 C CNN
@@
 $EndComp
 $Comp
-L DGND #PWR010
+L DGND #PWR08
 U 1 1 5281D360
 P 1900 2800
-AR Path="/5224C457/5281D330/5281D360" Ref="#PWR010"  Part="1"
-AR Path="/5224C457/5281E180/5281D360" Ref="#PWR019"  Part="1"
-AR Path="/5224C457/5281E2A4/5281D360" Ref="#PWR028"  Part="1"
-F 0 "#PWR010" H 1900 2800 40  0001 C CNN
+AR Path="/5224C457/5281D330/5281D360" Ref="#PWR08"  Part="1"
+AR Path="/5224C457/5281E180/5281D360" Ref="#PWR017"  Part="1"
+AR Path="/5224C457/5281E2A4/5281D360" Ref="#PWR026"  Part="1"
+F 0 "#PWR026" H 1900 2800 40  0001 C CNN
 F 1 "DGND" H 1900 2730 40  0000 C CNN
 F 2 "" H 1900 2800 60  0000 C CNN
@@
 $EndComp
 $Comp
-L +3.3V #PWR011
+L +3.3V #PWR09
 U 1 1 5281D366
 P 1900 1950
-AR Path="/5224C457/5281D330/5281D366" Ref="#PWR011"  Part="1"
-AR Path="/5224C457/5281E180/5281D366" Ref="#PWR020"  Part="1"
-AR Path="/5224C457/5281E2A4/5281D366" Ref="#PWR029"  Part="1"
-F 0 "#PWR011" H 1900 1910 30  0001 C CNN
+AR Path="/5224C457/5281D330/5281D366" Ref="#PWR09"  Part="1"
+AR Path="/5224C457/5281E180/5281D366" Ref="#PWR018"  Part="1"
+AR Path="/5224C457/5281E2A4/5281D366" Ref="#PWR027"  Part="1"
+F 0 "#PWR027" H 1900 1910 30  0001 C CNN
 F 1 "+3.3V" H 1900 2060 30  0000 C CNN
 F 2 "" H 1900 1950 60  0000 C CNN
@@
 AR Path="/5224C457/5281E180/5281D36C" Ref="R8"  Part="1"
 AR Path="/5224C457/5281E2A4/5281D36C" Ref="R13"  Part="1"
-F 0 "R3" V 3230 1950 40  0000 C CNN
+F 0 "R13" V 3230 1950 40  0000 C CNN
 F 1 "Nominal" V 3157 1951 40  0000 C CNN
 F 2 "~" V 3080 1950 30  0000 C CNN
@@
 AR Path="/5224C457/5281E180/5281D372" Ref="R9"  Part="1"
 AR Path="/5224C457/5281E2A4/5281D372" Ref="R14"  Part="1"
-F 0 "R4" V 3380 1950 40  0000 C CNN
+F 0 "R14" V 3380 1950 40  0000 C CNN
 F 1 "Nominal" V 3307 1951 40  0000 C CNN
 F 2 "~" V 3230 1950 30  0000 C CNN
@@
 $EndComp
 $Comp
-L +3.3V #PWR012
+L +3.3V #PWR010
 U 1 1 5281D378
 P 3150 1650
-AR Path="/5224C457/5281D330/5281D378" Ref="#PWR012"  Part="1"
-AR Path="/5224C457/5281E180/5281D378" Ref="#PWR021"  Part="1"
-AR Path="/5224C457/5281E2A4/5281D378" Ref="#PWR030"  Part="1"
-F 0 "#PWR012" H 3150 1610 30  0001 C CNN
+AR Path="/5224C457/5281D330/5281D378" Ref="#PWR010"  Part="1"
+AR Path="/5224C457/5281E180/5281D378" Ref="#PWR019"  Part="1"
+AR Path="/5224C457/5281E2A4/5281D378" Ref="#PWR028"  Part="1"
+F 0 "#PWR028" H 3150 1610 30  0001 C CNN
 F 1 "+3.3V" H 3150 1760 30  0000 C CNN
 F 2 "" H 3150 1650 60  0000 C CNN
@@
 AR Path="/5224C457/5281E180/5281D380" Ref="U24"  Part="1"
 AR Path="/5224C457/5281E2A4/5281D380" Ref="U27"  Part="1"
-F 0 "U21" H 4950 1350 60  0000 C CNN
+F 0 "U27" H 4950 1350 60  0000 C CNN
 F 1 "74LVC2G06" H 5100 1000 60  0000 C CNN
 F 2 "" H 4750 1050 60  0000 C CNN
@@
 AR Path="/5224C457/5281E180/5281D386" Ref="U24"  Part="2"
 AR Path="/5224C457/5281E2A4/5281D386" Ref="U27"  Part="2"
-F 0 "U21" H 6200 3400 60  0000 C CNN
+F 0 "U27" H 6200 3400 60  0000 C CNN
 F 1 "74LVC2G06" H 6350 3050 60  0000 C CNN
 F 2 "" H 6000 3100 60  0000 C CNN
@@
 $EndComp
 $Comp
-L DGND #PWR013
+L DGND #PWR011
 U 1 1 5281D38C
 P 4750 1450
-AR Path="/5224C457/5281D330/5281D38C" Ref="#PWR013"  Part="1"
-AR Path="/5224C457/5281E180/5281D38C" Ref="#PWR022"  Part="1"
-AR Path="/5224C457/5281E2A4/5281D38C" Ref="#PWR031"  Part="1"
-F 0 "#PWR013" H 4750 1450 40  0001 C CNN
+AR Path="/5224C457/5281D330/5281D38C" Ref="#PWR011"  Part="1"
+AR Path="/5224C457/5281E180/5281D38C" Ref="#PWR020"  Part="1"
+AR Path="/5224C457/5281E2A4/5281D38C" Ref="#PWR029"  Part="1"
+F 0 "#PWR029" H 4750 1450 40  0001 C CNN
 F 1 "DGND" H 4750 1380 40  0000 C CNN
 F 2 "" H 4750 1450 60  0000 C CNN
@@
 $EndComp
 $Comp
-L +3.3V #PWR014
+L +3.3V #PWR012
 U 1 1 5281D392
 P 4750 850
-AR Path="/5224C457/5281D330/5281D392" Ref="#PWR014"  Part="1"
-AR Path="/5224C457/5281E180/5281D392" Ref="#PWR023"  Part="1"
-AR Path="/5224C457/5281E2A4/5281D392" Ref="#PWR032"  Part="1"
-F 0 "#PWR014" H 4750 810 30  0001 C CNN
+AR Path="/5224C457/5281D330/5281D392" Ref="#PWR012"  Part="1"
+AR Path="/5224C457/5281E180/5281D392" Ref="#PWR021"  Part="1"
+AR Path="/5224C457/5281E2A4/5281D392" Ref="#PWR030"  Part="1"
+F 0 "#PWR030" H 4750 810 30  0001 C CNN
 F 1 "+3.3V" H 4750 960 30  0000 C CNN
 F 2 "" H 4750 850 60  0000 C CNN
@@
 AR Path="/5224C457/5281E180/5281D398" Ref="U26"  Part="1"
 AR Path="/5224C457/5281E2A4/5281D398" Ref="U29"  Part="1"
-F 0 "U23" H 4950 2350 60  0000 C CNN
+F 0 "U29" H 4950 2350 60  0000 C CNN
 F 1 "NC7WZ08" H 4950 2250 60  0000 C CNN
 F 2 "" H 4950 2300 60  0000 C CNN
@@
 AR Path="/5224C457/5281E180/5281D39E" Ref="U26"  Part="2"
 AR Path="/5224C457/5281E2A4/5281D39E" Ref="U29"  Part="2"
-F 0 "U23" H 4950 3250 60  0000 C CNN
+F 0 "U29" H 4950 3250 60  0000 C CNN
 F 1 "NC7WZ08" H 4950 3150 60  0000 C CNN
 F 2 "" H 4950 3200 60  0000 C CNN
@@
 NMOS_CTRL
 $Comp
-L DGND #PWR015
+L DGND #PWR013
 U 1 1 5281D3A6
 P 4750 2700
-AR Path="/5224C457/5281D330/5281D3A6" Ref="#PWR015"  Part="1"
-AR Path="/5224C457/5281E180/5281D3A6" Ref="#PWR024"  Part="1"
-AR Path="/5224C457/5281E2A4/5281D3A6" Ref="#PWR033"  Part="1"
-F 0 "#PWR015" H 4750 2700 40  0001 C CNN
+AR Path="/5224C457/5281D330/5281D3A6" Ref="#PWR013"  Part="1"
+AR Path="/5224C457/5281E180/5281D3A6" Ref="#PWR022"  Part="1"
+AR Path="/5224C457/5281E2A4/5281D3A6" Ref="#PWR031"  Part="1"
+F 0 "#PWR031" H 4750 2700 40  0001 C CNN
 F 1 "DGND" H 4750 2630 40  0000 C CNN
 F 2 "" H 4750 2700 60  0000 C CNN
@@
 $EndComp
 $Comp
-L +3.3V #PWR016
+L +3.3V #PWR014
 U 1 1 5281D3AC
 P 4750 1900
-AR Path="/5224C457/5281D330/5281D3AC" Ref="#PWR016"  Part="1"
-AR Path="/5224C457/5281E180/5281D3AC" Ref="#PWR025"  Part="1"
-AR Path="/5224C457/5281E2A4/5281D3AC" Ref="#PWR034"  Part="1"
-F 0 "#PWR016" H 4750 1860 30  0001 C CNN
+AR Path="/5224C457/5281D330/5281D3AC" Ref="#PWR014"  Part="1"
+AR Path="/5224C457/5281E180/5281D3AC" Ref="#PWR023"  Part="1"
+AR Path="/5224C457/5281E2A4/5281D3AC" Ref="#PWR032"  Part="1"
+F 0 "#PWR032" H 4750 1860 30  0001 C CNN
 F 1 "+3.3V" H 4750 2010 30  0000 C CNN
 F 2 "" H 4750 1900 60  0000 C CNN
@@
 AR Path="/5224C457/5281E180/5281D3B9" Ref="Q2"  Part="2"
 AR Path="/5224C457/5281E2A4/5281D3B9" Ref="Q3"  Part="2"
-F 0 "Q1" H 1700 651 40  0000 R CNN
+F 0 "Q3" H 1700 651 40  0000 R CNN
 F 1 "AON7611" H 1700 950 40  0000 R CNN
 F 2 "~" H 1570 902 29  0001 C CNN
@@
 AR Path="/5224C457/5281E180/5281D3BF" Ref="Q2"  Part="1"
 AR Path="/5224C457/5281E2A4/5281D3BF" Ref="Q3"  Part="1"
-F 0 "Q1" H 1300 651 40  0000 R CNN
+F 0 "Q3" H 1300 651 40  0000 R CNN
 F 1 "AON7611" H 1300 950 40  0000 R CNN
 F 2 "~" H 1170 902 29  0001 C CNN
@@
 AR Path="/5224C457/5281E180/5281D3C7" Ref="D3"  Part="1"
 AR Path="/5224C457/5281E2A4/5281D3C7" Ref="D5"  Part="1"
-F 0 "D1" H 1400 1450 40  0000 C CNN
+F 0 "D5" H 1400 1450 40  0000 C CNN
 F 1 "MBR1045ULPS" H 1400 1350 40  0000 C CNN
 F 2 "~" H 1400 1250 60  0000 C CNN
@@
 AR Path="/5224C457/5281E180/5281D3CD" Ref="D4"  Part="1"
 AR Path="/5224C457/5281E2A4/5281D3CD" Ref="D6"  Part="1"
-F 0 "D2" H 1600 1450 40  0000 C CNN
+F 0 "D6" H 1600 1450 40  0000 C CNN
 F 1 "MBR1045ULPS" H 1600 1350 40  0000 C CNN
 F 2 "~" H 1600 1250 60  0000 C CNN

Commit message: revisions to board and sch
Changed lines of the file:
@@
 $Descr A4 11693 8268
 encoding utf-8
-Sheet 3 15
+Sheet 3 16
 Title ""
-Date "18 jan 2014"
+Date "1 feb 2014"
 Rev ""
 Comp ""
@@
 AR Path="/5224C457/5281E180/5281D336" Ref="BT2"  Part="1"
 AR Path="/5224C457/5281E2A4/5281D336" Ref="BT3"  Part="1"
-F 0 "BT3" H 1300 2000 50  0000 C CNN
+F 0 "BT1" H 1300 2000 50  0000 C CNN
 F 1 "BATTERY" H 1300 1610 50  0000 C CNN
 F 2 "~" H 1300 1800 60  0000 C CNN
@@
 AR Path="/5224C457/5281E180/5281D33C" Ref="U25"  Part="1"
 AR Path="/5224C457/5281E2A4/5281D33C" Ref="U28"  Part="1"
-F 0 "U28" H 2450 2150 60  0000 C CNN
+F 0 "U22" H 2450 2150 60  0000 C CNN
 F 1 "TPS3700" H 2450 1550 60  0000 C CNN
 F 2 "" H 2450 2100 60  0000 C CNN
@@
 AR Path="/5224C457/5281E180/5281D342" Ref="R7"  Part="1"
 AR Path="/5224C457/5281E2A4/5281D342" Ref="R12"  Part="1"
-F 0 "R12" V 1780 1750 40  0000 C CNN
+F 0 "R2" V 1780 1750 40  0000 C CNN
 F 1 "1.58M" V 1707 1751 40  0000 C CNN
 F 2 "~" V 1630 1750 30  0000 C CNN
@@
 AR Path="/5224C457/5281E180/5281D348" Ref="R10"  Part="1"
 AR Path="/5224C457/5281E2A4/5281D348" Ref="R15"  Part="1"
-F 0 "R15" V 1780 2350 40  0000 C CNN
+F 0 "R5" V 1780 2350 40  0000 C CNN
 F 1 "102K" V 1707 2351 40  0000 C CNN
 F 2 "~" V 1630 2350 30  0000 C CNN
@@
 AR Path="/5224C457/5281E180/5281D34E" Ref="R11"  Part="1"
 AR Path="/5224C457/5281E2A4/5281D34E" Ref="R16"  Part="1"
-F 0 "R16" V 1780 2950 40  0000 C CNN
+F 0 "R6" V 1780 2950 40  0000 C CNN
 F 1 "191K" V 1707 2951 40  0000 C CNN
 F 2 "~" V 1630 2950 30  0000 C CNN
@@
 AR Path="/5224C457/5281E180/5281D354" Ref="#PWR015"  Part="1"
 AR Path="/5224C457/5281E2A4/5281D354" Ref="#PWR024"  Part="1"
-F 0 "#PWR024" H 1700 3250 40  0001 C CNN
+F 0 "#PWR06" H 1700 3250 40  0001 C CNN
 F 1 "DGND" H 1700 3180 40  0000 C CNN
 F 2 "" H 1700 3250 60  0000 C CNN
@@
 AR Path="/5224C457/5281E180/5281D35A" Ref="#PWR016"  Part="1"
 AR Path="/5224C457/5281E2A4/5281D35A" Ref="#PWR025"  Part="1"
-F 0 "#PWR025" H 1300 2150 40  0001 C CNN
+F 0 "#PWR07" H 1300 2150 40  0001 C CNN
 F 1 "DGND" H 1300 2080 40  0000 C CNN
 F 2 "" H 1300 2150 60  0000 C CNN
@@
 AR Path="/5224C457/5281E180/5281D360" Ref="#PWR017"  Part="1"
 AR Path="/5224C457/5281E2A4/5281D360" Ref="#PWR026"  Part="1"
-F 0 "#PWR026" H 1900 2800 40  0001 C CNN
+F 0 "#PWR08" H 1900 2800 40  0001 C CNN
 F 1 "DGND" H 1900 2730 40  0000 C CNN
 F 2 "" H 1900 2800 60  0000 C CNN
@@
 AR Path="/5224C457/5281E180/5281D366" Ref="#PWR018"  Part="1"
 AR Path="/5224C457/5281E2A4/5281D366" Ref="#PWR027"  Part="1"
-F 0 "#PWR027" H 1900 1910 30  0001 C CNN
+F 0 "#PWR09" H 1900 1910 30  0001 C CNN
 F 1 "+3.3V" H 1900 2060 30  0000 C CNN
 F 2 "" H 1900 1950 60  0000 C CNN
@@
 AR Path="/5224C457/5281E180/5281D36C" Ref="R8"  Part="1"
 AR Path="/5224C457/5281E2A4/5281D36C" Ref="R13"  Part="1"
-F 0 "R13" V 3230 1950 40  0000 C CNN
+F 0 "R3" V 3230 1950 40  0000 C CNN
 F 1 "Nominal" V 3157 1951 40  0000 C CNN
 F 2 "~" V 3080 1950 30  0000 C CNN
@@
 AR Path="/5224C457/5281E180/5281D372" Ref="R9"  Part="1"
 AR Path="/5224C457/5281E2A4/5281D372" Ref="R14"  Part="1"
-F 0 "R14" V 3380 1950 40  0000 C CNN
+F 0 "R4" V 3380 1950 40  0000 C CNN
 F 1 "Nominal" V 3307 1951 40  0000 C CNN
 F 2 "~" V 3230 1950 30  0000 C CNN
@@
 AR Path="/5224C457/5281E180/5281D378" Ref="#PWR019"  Part="1"
 AR Path="/5224C457/5281E2A4/5281D378" Ref="#PWR028"  Part="1"
-F 0 "#PWR028" H 3150 1610 30  0001 C CNN
+F 0 "#PWR010" H 3150 1610 30  0001 C CNN
 F 1 "+3.3V" H 3150 1760 30  0000 C CNN
 F 2 "" H 3150 1650 60  0000 C CNN
@@
 AR Path="/5224C457/5281E180/5281D380" Ref="U24"  Part="1"
 AR Path="/5224C457/5281E2A4/5281D380" Ref="U27"  Part="1"
-F 0 "U27" H 4950 1350 60  0000 C CNN
+F 0 "U21" H 4950 1350 60  0000 C CNN
 F 1 "74LVC2G06" H 5100 1000 60  0000 C CNN
 F 2 "" H 4750 1050 60  0000 C CNN
@@
 AR Path="/5224C457/5281E180/5281D386" Ref="U24"  Part="2"
 AR Path="/5224C457/5281E2A4/5281D386" Ref="U27"  Part="2"
-F 0 "U27" H 6200 3400 60  0000 C CNN
+F 0 "U21" H 6200 3400 60  0000 C CNN
 F 1 "74LVC2G06" H 6350 3050 60  0000 C CNN
 F 2 "" H 6000 3100 60  0000 C CNN
@@
 AR Path="/5224C457/5281E180/5281D38C" Ref="#PWR020"  Part="1"
 AR Path="/5224C457/5281E2A4/5281D38C" Ref="#PWR029"  Part="1"
-F 0 "#PWR029" H 4750 1450 40  0001 C CNN
+F 0 "#PWR011" H 4750 1450 40  0001 C CNN
 F 1 "DGND" H 4750 1380 40  0000 C CNN
 F 2 "" H 4750 1450 60  0000 C CNN
@@
 AR Path="/5224C457/5281E180/5281D392" Ref="#PWR021"  Part="1"
 AR Path="/5224C457/5281E2A4/5281D392" Ref="#PWR030"  Part="1"
-F 0 "#PWR030" H 4750 810 30  0001 C CNN
+F 0 "#PWR012" H 4750 810 30  0001 C CNN
 F 1 "+3.3V" H 4750 960 30  0000 C CNN
 F 2 "" H 4750 850 60  0000 C CNN
@@
 AR Path="/5224C457/5281E180/5281D398" Ref="U26"  Part="1"
 AR Path="/5224C457/5281E2A4/5281D398" Ref="U29"  Part="1"
-F 0 "U29" H 4950 2350 60  0000 C CNN
+F 0 "U23" H 4950 2350 60  0000 C CNN
 F 1 "NC7WZ08" H 4950 2250 60  0000 C CNN
 F 2 "" H 4950 2300 60  0000 C CNN
@@
 AR Path="/5224C457/5281E180/5281D39E" Ref="U26"  Part="2"
 AR Path="/5224C457/5281E2A4/5281D39E" Ref="U29"  Part="2"
-F 0 "U29" H 4950 3250 60  0000 C CNN
+F 0 "U23" H 4950 3250 60  0000 C CNN
 F 1 "NC7WZ08" H 4950 3150 60  0000 C CNN
 F 2 "" H 4950 3200 60  0000 C CNN
@@
 AR Path="/5224C457/5281E180/5281D3A6" Ref="#PWR022"  Part="1"
 AR Path="/5224C457/5281E2A4/5281D3A6" Ref="#PWR031"  Part="1"
-F 0 "#PWR031" H 4750 2700 40  0001 C CNN
+F 0 "#PWR013" H 4750 2700 40  0001 C CNN
 F 1 "DGND" H 4750 2630 40  0000 C CNN
 F 2 "" H 4750 2700 60  0000 C CNN
@@
 AR Path="/5224C457/5281E180/5281D3AC" Ref="#PWR023"  Part="1"
 AR Path="/5224C457/5281E2A4/5281D3AC" Ref="#PWR032"  Part="1"
-F 0 "#PWR032" H 4750 1860 30  0001 C CNN
+F 0 "#PWR014" H 4750 1860 30  0001 C CNN
 F 1 "+3.3V" H 4750 2010 30  0000 C CNN
 F 2 "" H 4750 1900 60  0000 C CNN
@@
 AR Path="/5224C457/5281E180/5281D3B9" Ref="Q2"  Part="2"
 AR Path="/5224C457/5281E2A4/5281D3B9" Ref="Q3"  Part="2"
-F 0 "Q3" H 1700 651 40  0000 R CNN
+F 0 "Q1" H 1700 651 40  0000 R CNN
 F 1 "AON7611" H 1700 950 40  0000 R CNN
 F 2 "~" H 1570 902 29  0001 C CNN
@@
 AR Path="/5224C457/5281E180/5281D3BF" Ref="Q2"  Part="1"
 AR Path="/5224C457/5281E2A4/5281D3BF" Ref="Q3"  Part="1"
-F 0 "Q3" H 1300 651 40  0000 R CNN
+F 0 "Q1" H 1300 651 40  0000 R CNN
 F 1 "AON7611" H 1300 950 40  0000 R CNN
 F 2 "~" H 1170 902 29  0001 C CNN
@@
 AR Path="/5224C457/5281E180/5281D3C7" Ref="D3"  Part="1"
 AR Path="/5224C457/5281E2A4/5281D3C7" Ref="D5"  Part="1"
-F 0 "D5" H 1400 1450 40  0000 C CNN
+F 0 "D1" H 1400 1450 40  0000 C CNN
 F 1 "MBR1045ULPS" H 1400 1350 40  0000 C CNN
 F 2 "~" H 1400 1250 60  0000 C CNN
@@
 AR Path="/5224C457/5281E180/5281D3CD" Ref="D4"  Part="1"
 AR Path="/5224C457/5281E2A4/5281D3CD" Ref="D6"  Part="1"
-F 0 "D6" H 1600 1450 40  0000 C CNN
+F 0 "D2" H 1600 1450 40  0000 C CNN
 F 1 "MBR1045ULPS" H 1600 1350 40  0000 C CNN
 F 2 "~" H 1600 1250 60  0000 C CNN
