File: interface_JTAG_2_wire.sch (KiCad schematic (older format))
At the start: 5 parts, among them U48 CONN_JTAG_14_2_wire

Commit message: placed components ... quite the task!
there is a lot of shit going on in this board... :D
Parts:
- renumbered C33 to C27, C34 to C28, C35 to C29, R51 to R46, U48 to U44
Changed lines of the file:
@@
 $Descr A4 11693 8268
 encoding utf-8
-Sheet 16 18
+Sheet 16 15
 Title ""
-Date "12 jan 2014"
+Date "18 jan 2014"
 Rev ""
 Comp ""
@@
 $EndDescr
 $Comp
-L CONN_JTAG_14 U48
+L CONN_JTAG_14 U44
 U 1 1 52A68398
 P 4450 2100
-F 0 "U48" H 4450 2100 60  0000 C CNN
+F 0 "U44" H 4450 2100 60  0000 C CNN
 F 1 "CONN_JTAG_14_2_wire" H 4450 1650 60  0000 C CNN
 F 2 "" H 4450 2100 60  0000 C CNN
@@
 $EndComp
 $Comp
-L C C33
+L C C27
 U 1 1 52A6994D
 P 4250 1000
-F 0 "C33" H 4250 1100 40  0000 L CNN
+F 0 "C27" H 4250 1100 40  0000 L CNN
 F 1 "0.1uF" H 4300 900 40  0000 L CNN
 F 2 "~" H 4288 850 30  0000 C CNN
@@
 $EndComp
 $Comp
-L +3.3V #PWR0111
+L +3.3V #PWR097
 U 1 1 52A69953
 P 4250 750
-F 0 "#PWR0111" H 4250 710 30  0001 C CNN
+F 0 "#PWR097" H 4250 710 30  0001 C CNN
 F 1 "+3.3V" H 4250 860 30  0000 C CNN
 F 2 "" H 4250 750 60  0000 C CNN
@@
 $EndComp
 $Comp
-L DGND #PWR0112
+L DGND #PWR098
 U 1 1 52A69959
 P 4250 1250
-F 0 "#PWR0112" H 4250 1250 40  0001 C CNN
+F 0 "#PWR098" H 4250 1250 40  0001 C CNN
 F 1 "DGND" H 4250 1180 40  0000 C CNN
 F 2 "" H 4250 1250 60  0000 C CNN
@@
 	4250 1200 4250 1250
 $Comp
-L +3.3V #PWR0113
+L +3.3V #PWR099
 U 1 1 52A69961
 P 3550 2150
-F 0 "#PWR0113" H 3550 2110 30  0001 C CNN
+F 0 "#PWR099" H 3550 2110 30  0001 C CNN
 F 1 "+3.3V" H 3550 2260 30  0000 C CNN
 F 2 "" H 3550 2150 60  0000 C CNN
@@
 	3550 2350 3650 2350
 $Comp
-L DGND #PWR0114
+L DGND #PWR0100
 U 1 1 52A69987
 P 3650 2550
-F 0 "#PWR0114" H 3650 2550 40  0001 C CNN
+F 0 "#PWR0100" H 3650 2550 40  0001 C CNN
 F 1 "DGND" H 3650 2480 40  0000 C CNN
 F 2 "" H 3650 2550 60  0000 C CNN
@@
 SBWTCK
 $Comp
-L CP1 C34
+L CP1 C28
 U 1 1 52A699A3
 P 4650 1000
-F 0 "C34" H 4700 1100 50  0000 L CNN
+F 0 "C28" H 4700 1100 50  0000 L CNN
 F 1 "10uF" H 4700 850 50  0000 L CNN
 F 2 "~" H 4650 1000 60  0000 C CNN
@@
 SBWTDIO
 $Comp
-L R R51
+L R R46
 U 1 1 52A69CB1
 P 5900 1900
-F 0 "R51" V 5980 1900 40  0000 C CNN
+F 0 "R46" V 5980 1900 40  0000 C CNN
 F 1 "47K" V 5907 1901 40  0000 C CNN
 F 2 "~" V 5830 1900 30  0000 C CNN
@@
 $EndComp
 $Comp
-L C C35
+L C C29
 U 1 1 52A69CB7
 P 5900 2550
-F 0 "C35" H 5900 2650 40  0000 L CNN
+F 0 "C29" H 5900 2650 40  0000 L CNN
 F 1 "2.2 nF" H 5950 2450 40  0000 L CNN
 F 2 "~" H 5938 2400 30  0000 C CNN
@@
 Connection ~ 5900 2250
 $Comp
-L +3.3V #PWR0115
+L +3.3V #PWR0101
 U 1 1 52A69CDC
 P 5900 1600
-F 0 "#PWR0115" H 5900 1560 30  0001 C CNN
+F 0 "#PWR0101" H 5900 1560 30  0001 C CNN
 F 1 "+3.3V" H 5900 1710 30  0000 C CNN
 F 2 "" H 5900 1600 60  0000 C CNN
@@
 	5900 1600 5900 1650
 $Comp
-L DGND #PWR0116
+L DGND #PWR0102
 U 1 1 52A69CF0
 P 5900 2800
-F 0 "#PWR0116" H 5900 2800 40  0001 C CNN
+F 0 "#PWR0102" H 5900 2800 40  0001 C CNN
 F 1 "DGND" H 5900 2730 40  0000 C CNN
 F 2 "" H 5900 2800 60  0000 C CNN
