File: signal_leds.sch (KiCad schematic (older format))
At the start: 10 parts

Commit message: replacement of parts, moved parts, preparing for routing
Changed lines of the file:
@@
 Sheet 10 16
 Title ""
-Date "1 feb 2014"
+Date "3 feb 2014"
 Rev ""
 Comp ""
@@
 AR Path="/52A0B607/52E619E4/52E6286C" Ref="R7"  Part="1"
 AR Path="/52A0B607/52ECD75E/52E6286C" Ref="R12"  Part="1"
-F 0 "R7" V 6430 3950 40  0000 C CNN
+F 0 "R12" V 6430 3950 40  0000 C CNN
 F 1 "200" V 6357 3951 40  0000 C CNN
 F 2 "~" V 6280 3950 30  0000 C CNN
@@
 AR Path="/52A0B607/52E619E4/52E62872" Ref="D6"  Part="1"
 AR Path="/52A0B607/52ECD75E/52E62872" Ref="D26"  Part="1"
-F 0 "D6" H 5800 4100 50  0000 C CNN
+F 0 "D26" H 5800 4100 50  0000 C CNN
 F 1 "LY-A67F" H 5800 3800 50  0001 C CNN
 F 2 "~" H 5800 4000 60  0000 C CNN
@@
 AR Path="/52A0B607/52E619E4/52E62878" Ref="D10"  Part="1"
 AR Path="/52A0B607/52ECD75E/52E62878" Ref="D27"  Part="1"
-F 0 "D10" H 6100 4100 50  0000 C CNN
+F 0 "D27" H 6100 4100 50  0000 C CNN
 F 1 "LY-A67F" H 6100 3800 50  0001 C CNN
 F 2 "~" H 6100 4000 60  0000 C CNN
@@
 AR Path="/52A0B607/52E619E4/52E6287E" Ref="D5"  Part="1"
 AR Path="/52A0B607/52ECD75E/52E6287E" Ref="D25"  Part="1"
-F 0 "D5" H 5350 3850 50  0000 C CNN
+F 0 "D25" H 5350 3850 50  0000 C CNN
 F 1 "LY-E63F" H 5350 3550 50  0001 C CNN
 F 2 "~" H 5350 3750 60  0000 C CNN
@@
 AR Path="/52A0B607/52E619E4/52E62884" Ref="D13"  Part="1"
 AR Path="/52A0B607/52ECD75E/52E62884" Ref="D30"  Part="1"
-F 0 "D13" H 5200 4200 50  0000 C CNN
+F 0 "D30" H 5200 4200 50  0000 C CNN
 F 1 "LY-E63F" H 5200 3900 50  0001 C CNN
 F 2 "~" H 5200 4100 60  0000 C CNN
@@
 AR Path="/52A0B607/52E619E4/52E6288A" Ref="D4"  Part="1"
 AR Path="/52A0B607/52ECD75E/52E6288A" Ref="D24"  Part="1"
-F 0 "D4" H 5050 3850 50  0000 C CNN
+F 0 "D24" H 5050 3850 50  0000 C CNN
 F 1 "LY-E63F" H 5050 3550 50  0001 C CNN
 F 2 "~" H 5050 3750 60  0000 C CNN
@@
 AR Path="/52A0B607/52E619E4/52E62890" Ref="D12"  Part="1"
 AR Path="/52A0B607/52ECD75E/52E62890" Ref="D29"  Part="1"
-F 0 "D12" H 4900 4200 50  0000 C CNN
+F 0 "D29" H 4900 4200 50  0000 C CNN
 F 1 "LY-E63F" H 4900 3900 50  0001 C CNN
 F 2 "~" H 4900 4100 60  0000 C CNN
@@
 AR Path="/52A0B607/52E619E4/52E62896" Ref="D3"  Part="1"
 AR Path="/52A0B607/52ECD75E/52E62896" Ref="D23"  Part="1"
-F 0 "D3" H 4750 3850 50  0000 C CNN
+F 0 "D23" H 4750 3850 50  0000 C CNN
 F 1 "LY-E63F" H 4750 3550 50  0001 C CNN
 F 2 "~" H 4750 3750 60  0000 C CNN
@@
 AR Path="/52A0B607/52E619E4/52E6289C" Ref="D11"  Part="1"
 AR Path="/52A0B607/52ECD75E/52E6289C" Ref="D28"  Part="1"
-F 0 "D11" H 4600 4200 50  0000 C CNN
+F 0 "D28" H 4600 4200 50  0000 C CNN
 F 1 "LY-E63F" H 4600 3900 50  0001 C CNN
 F 2 "~" H 4600 4100 60  0000 C CNN
@@
 AR Path="/52A0B607/52E619E4/52ECA2F4" Ref="D14"  Part="1"
 AR Path="/52A0B607/52ECD75E/52ECA2F4" Ref="D31"  Part="1"
-F 0 "D14" H 5500 4200 50  0000 C CNN
+F 0 "D31" H 5500 4200 50  0000 C CNN
 F 1 "LY-E63F" H 5500 3900 50  0001 C CNN
 F 2 "~" H 5500 4100 60  0000 C CNN
