File: sensors_touch.sch (KiCad schematic (older format))
At the start: 21 parts, among them U33 AT42QT1011, U34 TOUCHPAD, U35 AT42QT1011, U36 TOUCHPAD, U37 AT42QT1011, U38 TOUCHPAD

Commit message: began routing!!!!!
:D
gonna try the autorouter after important traces.
Parts:
- added P10, P11, P12, P13, P14, P15, P16, P7, P8, P9: CONN_2, ~, symbol CONN_2
Connections:
- net +3.3V: now also P14.2 (PM), P9.2 (PM)
- net DGND: now also P11.2 (PM), P16.2 (PM)
- net TOUCH_1: now also P14.1 (P1), P9.1 (P1)
- net TOUCH_2: now also P10.1 (P1), P15.1 (P1)
- net TOUCH_3: now also P11.1 (P1), P16.1 (P1)
- no-connect marks 0 -> 10
Other:
- note added: "Linkages to main board"
Changed lines of the file:
@@
 Sheet 7 16
 Title ""
-Date "8 feb 2014"
+Date "10 feb 2014"
 Rev ""
 Comp ""
@@
 	1    0    0    -1
 $EndComp
+$Comp
+L CONN_2 P7
+U 1 1 52F869B3
+P 5250 1000
+F 0 "P7" V 5200 1000 40  0000 C CNN
+F 1 "CONN_2" V 5300 1000 40  0000 C CNN
+F 2 "~" H 5250 1000 60  0000 C CNN
+F 3 "~" H 5250 1000 60  0000 C CNN
+	1    5250 1000
+	1    0    0    -1
+$EndComp
+$Comp
+L CONN_2 P8
+U 1 1 52F869C0
+P 5250 1400
+F 0 "P8" V 5200 1400 40  0000 C CNN
+F 1 "CONN_2" V 5300 1400 40  0000 C CNN
+F 2 "~" H 5250 1400 60  0000 C CNN
+F 3 "~" H 5250 1400 60  0000 C CNN
+	1    5250 1400
+	1    0    0    -1
+$EndComp
+$Comp
+L CONN_2 P9
+U 1 1 52F869C6
+P 5250 2050
+F 0 "P9" V 5200 2050 40  0000 C CNN
+F 1 "CONN_2" V 5300 2050 40  0000 C CNN
+F 2 "~" H 5250 2050 60  0000 C CNN
+F 3 "~" H 5250 2050 60  0000 C CNN
+	1    5250 2050
+	1    0    0    -1
+$EndComp
+$Comp
+L CONN_2 P10
+U 1 1 52F869CC
+P 5250 2450
+F 0 "P10" V 5200 2450 40  0000 C CNN
+F 1 "CONN_2" V 5300 2450 40  0000 C CNN
+F 2 "~" H 5250 2450 60  0000 C CNN
+F 3 "~" H 5250 2450 60  0000 C CNN
+	1    5250 2450
+	1    0    0    -1
+$EndComp
+$Comp
+L CONN_2 P11
+U 1 1 52F869D2
+P 5250 2850
+F 0 "P11" V 5200 2850 40  0000 C CNN
+F 1 "CONN_2" V 5300 2850 40  0000 C CNN
+F 2 "~" H 5250 2850 60  0000 C CNN
+F 3 "~" H 5250 2850 60  0000 C CNN
+	1    5250 2850
+	1    0    0    -1
+$EndComp
+Text HLabel 4800 1950 0    60   Output ~ 0
+TOUCH_1
+Text HLabel 4800 2350 0    60   Output ~ 0
+TOUCH_2
+Text HLabel 4800 2750 0    60   Output ~ 0
+TOUCH_3
+Wire Wire Line
+	4800 1950 4900 1950
+Wire Wire Line
+	4800 2350 4900 2350
+Wire Wire Line
+	4800 2750 4900 2750
+Wire Wire Line
+	4900 900  4800 900
+Wire Wire Line
+	4800 1100 4900 1100
+Wire Wire Line
+	4900 1300 4800 1300
+Wire Wire Line
+	4800 1500 4900 1500
+NoConn ~ 4800 900
+NoConn ~ 4800 1100
+NoConn ~ 4800 1300
+NoConn ~ 4800 1500
+$Comp
+L DGND #PWR041
+U 1 1 52F86C74
+P 4800 3050
+F 0 "#PWR041" H 4800 3050 40  0001 C CNN
+F 1 "DGND" H 4800 2980 40  0000 C CNN
+F 2 "" H 4800 3050 60  0000 C CNN
+F 3 "" H 4800 3050 60  0000 C CNN
+	1    4800 3050
+	1    0    0    -1
+$EndComp
+Wire Wire Line
+	4900 2950 4800 2950
+Wire Wire Line
+	4800 2950 4800 3050
+$Comp
+L +3.3V #PWR042
+U 1 1 52F86CD3
+P 4800 2150
+F 0 "#PWR042" H 4800 2110 30  0001 C CNN
+F 1 "+3.3V" H 4800 2260 30  0000 C CNN
+F 2 "" H 4800 2150 60  0000 C CNN
+F 3 "" H 4800 2150 60  0000 C CNN
+	1    4800 2150
+	1    0    0    -1
+$EndComp
+Wire Wire Line
+	4800 2150 4900 2150
+Wire Wire Line
+	4900 2550 4800 2550
+NoConn ~ 4800 2550
+Wire Notes Line
+	5400 700  5600 700
+Wire Notes Line
+	5500 700  5500 3100
+Wire Notes Line
+	5400 3100 5600 3100
+Text Notes 5000 650  0    60   ~ 0
+Linkages to main board
+$Comp
+L CONN_2 P12
+U 1 1 52F87534
+P 5800 1000
+F 0 "P12" V 5750 1000 40  0000 C CNN
+F 1 "CONN_2" V 5850 1000 40  0000 C CNN
+F 2 "~" H 5800 1000 60  0000 C CNN
+F 3 "~" H 5800 1000 60  0000 C CNN
+	1    5800 1000
+	-1   0    0    -1
+$EndComp
+$Comp
+L CONN_2 P13
+U 1 1 52F8753A
+P 5800 1400
+F 0 "P13" V 5750 1400 40  0000 C CNN
+F 1 "CONN_2" V 5850 1400 40  0000 C CNN
+F 2 "~" H 5800 1400 60  0000 C CNN
+F 3 "~" H 5800 1400 60  0000 C CNN
+	1    5800 1400
+	-1   0    0    -1
+$EndComp
+$Comp
+L CONN_2 P14
+U 1 1 52F87540
+P 5800 2050
+F 0 "P14" V 5750 2050 40  0000 C CNN
+F 1 "CONN_2" V 5850 2050 40  0000 C CNN
+F 2 "~" H 5800 2050 60  0000 C CNN
+F 3 "~" H 5800 2050 60  0000 C CNN
+	1    5800 2050
+	-1   0    0    -1
+$EndComp
+$Comp
+L CONN_2 P15
+U 1 1 52F87546
+P 5800 2450
+F 0 "P15" V 5750 2450 40  0000 C CNN
+F 1 "CONN_2" V 5850 2450 40  0000 C CNN
+F 2 "~" H 5800 2450 60  0000 C CNN
+F 3 "~" H 5800 2450 60  0000 C CNN
+	1    5800 2450
+	-1   0    0    -1
+$EndComp
+$Comp
+L CONN_2 P16
+U 1 1 52F8754C
+P 5800 2850
+F 0 "P16" V 5750 2850 40  0000 C CNN
+F 1 "CONN_2" V 5850 2850 40  0000 C CNN
+F 2 "~" H 5800 2850 60  0000 C CNN
+F 3 "~" H 5800 2850 60  0000 C CNN
+	1    5800 2850
+	-1   0    0    -1
+$EndComp
+Text HLabel 6250 1950 2    60   Output ~ 0
+TOUCH_1
+Text HLabel 6250 2350 2    60   Output ~ 0
+TOUCH_2
+Text HLabel 6250 2750 2    60   Output ~ 0
+TOUCH_3
+Wire Wire Line
+	6250 1950 6150 1950
+Wire Wire Line
+	6250 2350 6150 2350
+Wire Wire Line
+	6250 2750 6150 2750
+Wire Wire Line
+	6150 900  6250 900
+Wire Wire Line
+	6250 1100 6150 1100
+Wire Wire Line
+	6150 1300 6250 1300
+Wire Wire Line
+	6250 1500 6150 1500
+NoConn ~ 6250 900
+NoConn ~ 6250 1100
+NoConn ~ 6250 1300
+NoConn ~ 6250 1500
+$Comp
+L DGND #PWR043
+U 1 1 52F87560
+P 6250 3050
+F 0 "#PWR043" H 6250 3050 40  0001 C CNN
+F 1 "DGND" H 6250 2980 40  0000 C CNN
+F 2 "" H 6250 3050 60  0000 C CNN
+F 3 "" H 6250 3050 60  0000 C CNN
+	1    6250 3050
+	-1   0    0    -1
+$EndComp
+Wire Wire Line
+	6150 2950 6250 2950
+Wire Wire Line
+	6250 2950 6250 3050
+$Comp
+L +3.3V #PWR044
+U 1 1 52F87568
+P 6250 2150
+F 0 "#PWR044" H 6250 2110 30  0001 C CNN
+F 1 "+3.3V" H 6250 2260 30  0000 C CNN
+F 2 "" H 6250 2150 60  0000 C CNN
+F 3 "" H 6250 2150 60  0000 C CNN
+	1    6250 2150
+	-1   0    0    -1
+$EndComp
+Wire Wire Line
+	6250 2150 6150 2150
+Wire Wire Line
+	6150 2550 6250 2550
+NoConn ~ 6250 2550
 $EndSCHEMATC
